Commit message: Project building and running but controller not working

File: canopen_tests/urdf/eirabot_controller/robot_controller.macro.xacro (robot description, xacro)
@@ -44,5 +44,5 @@
         <child link="${prefix}link1"/>
     </joint>
-    <joint name="${prefix}joint1" type="revolute">
+    <joint name="${prefix}joint_1" type="revolute">
         <parent link="${prefix}link1"/>
         <child link="${prefix}link2"/>
@@ -51,5 +51,5 @@
         <limit lower="${-2*pi}" upper="${2*pi}" effort="10.0" velocity="0.5"/>
     </joint>
-    <joint name="${prefix}joint2" type="revolute">
+    <joint name="${prefix}joint_2" type="revolute">
         <parent link="${prefix}link2"/>
         <child link="${prefix}link3"/>
@@ -58,5 +58,5 @@
         <limit lower="${-2*pi}" upper="${2*pi}" effort="10.0" velocity="0.5"/>
     </joint>
-    <joint name="${prefix}joint3" type="fixed">
+    <joint name="${prefix}joint_3" type="fixed">
         <parent link="${prefix}link3"/>
         <child link="${prefix}link4"/>

File: canopen_tests/urdf/eirabot_controller/robot_controller.ros2_control.xacro (robot description, xacro)
@@ -16,10 +16,12 @@
               <param name="master_bin">"${master_bin}"</param>
             </hardware>
-            <joint name="${prefix}joint1">
+            <joint name="${prefix}joint_1">
                 <param name="device_name">joint_1</param>
+                <command_interface name="velocity"/>
                 <state_interface name="position" />
             </joint>
-            <joint name="${prefix}joint2">
+            <joint name="${prefix}joint_2">
                 <param name="device_name">joint_2</param>
+                <command_interface name="velocity"/>
                 <state_interface name="position" />
             </joint>
