Commit message: Updated urdf files to diff drive rather than robot arm

File: canopen_tests/urdf/eirabot_controller/robot_controller.ros2_control.xacro (robot description, xacro)
@@ -16,12 +16,10 @@
               <param name="master_bin">"${master_bin}"</param>
             </hardware>
-            <joint name="${prefix}joint_1">
-                <param name="device_name">joint_1</param>
-                <command_interface name="velocity"/>
+            <joint name="${prefix}left_wheel_joint">
+                <param name="device_name">left_wheel_joint</param>
                 <state_interface name="position" />
             </joint>
-            <joint name="${prefix}joint_2">
-                <param name="device_name">joint_2</param>
-                <command_interface name="velocity"/>
+            <joint name="${prefix}right_wheel_joint">
+                <param name="device_name">right_wheel_joint</param>
                 <state_interface name="position" />
             </joint>

File: canopen_tests/urdf/eirabot_controller/robot_controller.urdf.xacro (robot description, xacro)
@@ -1,19 +1,16 @@
 <?xml version="1.0"?>
 <robot xmlns:xacro="http://wiki.ros.org/xacro" name="test_robot">
-    <xacro:include filename="$(find canopen_tests)/urdf/robot_controller/robot_controller.macro.xacro"/>
-    <xacro:include filename="$(find canopen_tests)/urdf/robot_controller/robot_controller.ros2_control.xacro"/>
-    <link name="world" />
-    <xacro:robot_control_robot
-        name="test_robot"
+    <xacro:include filename="$(find canopen_tests)/urdf/eirabot_controller/diffbot.materials.xacro"/>
+    <xacro:include filename="$(find canopen_tests)/urdf/eirabot_controller/diffbot_description.urdf.xacro"/>
+    <!--<xacro:include filename="$(find canopen_tests)/urdf/eirabot_controller/robot_controller.macro.xacro"/>-->
+    <xacro:include filename="$(find canopen_tests)/urdf/eirabot_controller/robot_controller.ros2_control.xacro"/>
+    <xacro:diffbot
         prefix=""
-        parent="world"
-        >
-            <origin xyz="0 0 0" rpy="0 0 0" />
-    </xacro:robot_control_robot>
+        />
     <xacro:robot_control_control
         name="test_robot"
         prefix=""
-        bus_config="$(find canopen_tests)/config/robot_control/bus.yml"
-        master_config="$(find canopen_tests)/config/robot_control/master.dcf"
+        bus_config="$(find canopen_tests)/config/eirabot_control/bus.yml"
+        master_config="$(find canopen_tests)/config/eirabot_control/master.dcf"
         can_interface_name="can0"
         master_bin="" />
